File: Modbus-RJ45-Breakout.kicad_pcb (KiCad board)
At the start: 2 copper layers, 86 x 68 mm, 86 parts, among them J1 RJ45_Weidmueller_2562920000, J10 USB_B_Mini, J2 RJ45_Weidmueller_2562920000, J3 Conn_01x04, J4 Conn_01x04, J5 Conn_01x02, J6 Conn_01x02, J7 Conn_01x02, J8 Conn_01x02, J9 USB_B_Mini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

Commit message: Added the revision license and author information
Routing:
- net GNDS: vias 46 -> 42
- net GND1: vias 55 -> 54
Other:
- board text added: "${COMPANY} - ${COMMENT1} ${TITLE} ${REVISION}"
Changed lines of the file:
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@@
   )
   (paper "A4")
+  (title_block
+    (title "Modbus-RJ45-Breakout")
+    (date "2023-04-24")
+    (rev "0.0.1")
+    (company "the78mole")
+    (comment 1 "Daniel Glaser")
+  )
   (layers
     (0 "F.Cu" signal)
@@
   (gr_rect (start 50 50) (end 136 118) (layer "Edge.Cuts") (width 0.1) (fill none))
   (gr_rect (start 50 50) (end 136 118) (layer "Margin") (width 0.15) (fill none))
+  (gr_text "${COMPANY} - ${COMMENT1}\n${TITLE} \n${REVISION} \n" (at 116.65 69.2) (layer "F.Mask")
+    (effects (font (size 1 1) (thickness 0.15)))
+  )
   (segment (start 127.3 62.5) (end 127.4 62.4) (width 1) (layer "F.Cu") (net 1))
   (segment (start 132.9 53.6) (end 132.9 62.4) (width 1) (layer "F.Cu") (net 1))
@@
   (via (at 112 63.25) (size 0.8) (drill 0.4) (layers "F.Cu" "B.Cu") (free) (net 2))
   (via (at 134 81.75) (size 0.8) (drill 0.4) (layers "F.Cu" "B.Cu") (free) (net 2))
-  (via (at 114 66) (size 0.8) (drill 0.4) (layers "F.Cu" "B.Cu") (free) (net 2))
+  (via (at 114.1 65.5) (size 0.8) (drill 0.4) (layers "F.Cu" "B.Cu") (free) (net 2))
   (via (at 117 75.25) (size 0.8) (drill 0.4) (layers "F.Cu" "B.Cu") (free) (net 2))
-  (via (at 108.25 67) (size 0.8) (drill 0.4) (layers "F.Cu" "B.Cu") (free) (net 2))
   (via (at 134 76) (size 0.8) (drill 0.4) (layers "F.Cu" "B.Cu") (free) (net 2))
   (via (at 101.75 52.25) (size 0.8) (drill 0.4) (layers "F.Cu" "B.Cu") (free) (net 2))
@@
   (via (at 85 61.25) (size 0.8) (drill 0.4) (layers "F.Cu" "B.Cu") (free) (net 2))
   (via (at 114.5 78.25) (size 0.8) (drill 0.4) (layers "F.Cu" "B.Cu") (free) (net 2))
-  (via (at 125.5 67) (size 0.8) (drill 0.4) (layers "F.Cu" "B.Cu") (free) (net 2))
+  (via (at 124.85 65.85) (size 0.8) (drill 0.4) (layers "F.Cu" "B.Cu") (free) (net 2))
   (via (at 133.75 65.25) (size 0.8) (drill 0.4) (layers "F.Cu" "B.Cu") (free) (net 2))
   (via (at 104 72.5) (size 0.8) (drill 0.4) (layers "F.Cu" "B.Cu") (free) (net 2))
@@
   (segment (start 101.5 108.25) (end 102.2 107.55) (width 0.2) (layer "B.Cu") (net 43))
   (segment (start 74.25 100.5) (end 74.25 69.25) (width 0.5) (layer "F.Cu") (net 45))
-  (via (at 67 59.25) (size 0.8) (drill 0.4) (layers "F.Cu" "B.Cu") (free) (net 45))
   (via (at 66.5 84) (size 0.8) (drill 0.4) (layers "F.Cu" "B.Cu") (free) (net 45))
   (via (at 61.75 68.5) (size 0.8) (drill 0.4) (layers "F.Cu" "B.Cu") (free) (net 45))
@@
   (via (at 68.75 67.5) (size 0.8) (drill 0.4) (layers "F.Cu" "B.Cu") (free) (net 45))
   (via (at 58.75 95) (size 0.8) (drill 0.4) (layers "F.Cu" "B.Cu") (free) (net 45))
-  (via (at 74.25 57.75) (size 0.8) (drill 0.4) (layers "F.Cu" "B.Cu") (free) (net 45))
   (via (at 59 68.75) (size 0.8) (drill 0.4) (layers "F.Cu" "B.Cu") (free) (net 45))
   (via (at 75.5 77.75) (size 0.8) (drill 0.4) (layers "F.Cu" "B.Cu") (free) (net 45))
@@
   (via (at 75.5 70.75) (size 0.8) (drill 0.4) (layers "F.Cu" "B.Cu") (free) (net 45))
   (via (at 51.75 116.25) (size 0.8) (drill 0.4) (layers "F.Cu" "B.Cu") (free) (net 45))
-  (via (at 62.75 57.75) (size 0.8) (drill 0.4) (layers "F.Cu" "B.Cu") (free) (net 45))
   (via (at 52.5 92.75) (size 0.8) (drill 0.4) (layers "F.Cu" "B.Cu") (free) (net 45))
   (via (at 52.5 101) (size 0.8) (drill 0.4) (layers "F.Cu" "B.Cu") (free) (net 45))
@@
   (via (at 53 62.75) (size 0.8) (drill 0.4) (layers "F.Cu" "B.Cu") (free) (net 45))
   (via (at 52 51.75) (size 0.8) (drill 0.4) (layers "F.Cu" "B.Cu") (free) (net 45))
-  (via (at 59.25 62) (size 0.8) (drill 0.4) (layers "F.Cu" "B.Cu") (free) (net 45))
   (via (at 54.75 106) (size 0.8) (drill 0.4) (layers "F.Cu" "B.Cu") (free) (net 45))
   (via (at 75.25 94.75) (size 0.8) (drill 0.4) (layers "F.Cu" "B.Cu") (free) (net 45))
