File: Modbus-RJ45-Breakout.kicad_pcb (KiCad board)
At the start: 2 copper layers, 86 x 68 mm, 86 parts, among them J1 RJ45_Weidmueller_2562920000, J10 USB_B_Mini, J2 RJ45_Weidmueller_2562920000, J3 Conn_01x04, J4 Conn_01x04, J5 Conn_01x02, J6 Conn_01x02, J7 Conn_01x02, J8 Conn_01x02, J9 USB_B_Mini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

Commit message: Added some 3D shapes -> Ethernet Connectors wrong
Parts:
- J10, J9: footprint Connector_USB:USB_Mini-B_Wuerth_65100516121_Horizontal -> the78mole:USB_Mini-B_Wuerth_65100516121_Horizontal
- J3, J4: footprint Connector_Wago:Wago_734-164_1x04_P3.50mm_Horizontal -> the78mole:Wago_734-164_1x04_P3.50mm_Horizontal
- U3, U8: footprint Package_SO:SO-8_3.9x4.9mm_P1.27mm -> the78mole:SO-8_3.9x4.9mm_P1.27mm
