File: Modbus-RJ45-Breakout.kicad_sch (KiCad schematic)
At the start: 22 parts, among them J1 RJ45_Weidmueller_2562920000, J2 RJ45_Weidmueller_2562920000, J3 Conn_01x04, J4 Conn_01x04, J5 Conn_01x02, J6 Conn_01x02, J7 Conn_01x02, J8 Conn_01x02

Commit message: Added the revision license and author information
Parts:
- R2, R3: value (none) -> 560; footprint (none) -> Resistor_SMD:R_0603_1608Metric_Pad0.98x0.95mm_HandSolder
Other:
- company: (none) -> the78mole
- title: (none) -> Modbus-RJ45-Breakout
Changed lines of the file:
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@@
 (kicad_sch (version 20211123) (generator eeschema)
   (paper "A4")
+  (title_block
+    (title "Modbus-RJ45-Breakout")
+    (date "2023-04-24")
+    (rev "0.0.1")
+    (company "the78mole")
+  )
   (junction (at 192.405 60.325) (diameter 0) (color 0 0 0 0)
   )
@@
     (in_bom yes) (on_board yes)
     (property "Reference" "R3" (id 0) (at 225.425 72.39 90))
-    (property "Value" "" (id 1) (at 220.98 72.39 90))
-    (property "Footprint" "" (id 2) (at 222.885 72.39 0)
+    (property "Value" "560" (id 1) (at 220.98 72.39 90))
+    (property "Footprint" "Resistor_SMD:R_0603_1608Metric_Pad0.98x0.95mm_HandSolder" (id 2) (at 222.885 72.39 0)
       (effects (font (size 1.27 1.27)) hide)
     )
@@
     (in_bom yes) (on_board yes)
     (property "Reference" "R2" (id 0) (at 225.425 38.1 90))
-    (property "Value" "" (id 1) (at 220.98 38.1 90))
-    (property "Footprint" "" (id 2) (at 222.885 38.1 0)
-      (effects (font (size 1.27 1.27)) hide)
-    )
+    (property "Value" "560" (id 1) (at 220.98 38.1 90))
+    (property "Footprint" "Resistor_SMD:R_0603_1608Metric_Pad0.98x0.95mm_HandSolder" (id 2) (at 222.885 38.1 0)
+      (effects (font (size 1.27 1.27)) hide)
+    )
